Commit message: :sparkles: Update models

File: res/urdf/orange_cup.urdf (robot description, URDF)
Before this commit: robot orange_cup, 1 links, 0 joints
Links:
- link orange_cup: geometry collision mesh filename=package://laas_objects/res/obj/orange_cup.obj; visual mesh filename=package://laas_objects/res/obj/orange_cup.obj

File: res/urdf/red_ball.urdf (robot description, URDF)
Before this commit: robot red_ball, 1 links, 0 joints
Links:
- link red_ball: geometry collision mesh filename=package://laas_objects/res/obj/red_ball.obj; visual mesh filename=package://laas_objects/res/obj/red_ball.obj
