Commit message: :tada: new objects

File: res/urdf/blue_bin.urdf (robot description, URDF)
Before this commit: robot blue_bin, 1 links, 0 joints
Links:
- link blue_bin: mass 0.5 -> 0.7

File: res/urdf/green_bin.urdf (robot description, URDF)
Before this commit: robot green_bin, 1 links, 0 joints
Links:
- link green_bin: mass 0.5 -> 0.7; geometry collision box size=0.27 0.3 0.005; collision box size=0.27 0.3 0.005

File: res/urdf/orange_cup.urdf (robot description, URDF)
Before this commit: robot orange_cup, 1 links, 0 joints
Links:
- link orange_cup: mass 0.075 -> 0.15

File: res/urdf/plane.urdf (robot description, URDF)
Before this commit: robot plane, 1 links, 0 joints
Links:
- link planeLink: geometry collision box size=200 200 0.001; visual mesh filename=package://laas_objects/res/obj/plane.obj scale=1 1 1

Commit message: :sparkles: new objects added 	modifié :         launch/cup_stack_detector.launch 	modifié :         launch/cup_stack_provider.launch 	nouveau fichier : launch/iros2019_detector.launch 	nouveau fichier : launch/iros2019_provider.launch 	modifié :         res/blend/adream_empty.blend 	modifié :         res/blend/green_bin.blend 	nouveau fichier : res/blend/green_bin.blend1 	nouveau fichier : res/blend/green_cylinder.blend 	modifié :         res/blend/orange_cup.blend 	nouveau fichier : res/blend/orange_cup.blend1 	nouveau fichier : res/blend/yellow_ball.blend 	modifié :         res/obj/green_bin.obj 	nouveau fichier : res/obj/green_cylinder.mtl 	nouveau fichier : res/obj/green_cylinder.obj 	renommé :         res/obj/IKEA_table_TORSBY.mtl -> res/obj/table.mtl 	renommé :         res/obj/IKEA_table_TORSBY.obj -> res/obj/table.obj 	modifié :         res/tags/blue_bin.xml 	modifié :         res/tags/green_bin.xml 	modifié :         res/urdf/blue_bin.urdf 	modifié :         res/urdf/green_bin.urdf 	nouveau fichier : res/urdf/green_cylinder.urdf 	modifié :         res/urdf/orange_cup.urdf 	modifié :         res/urdf/plane.urdf 	modifié :         res/urdf/red_cup.urdf 	renommé :         res/urdf/IKEA_table_TORSBY.urdf -> res/urdf/table.urdf 	supprimé :        res/urdf/wallsi.urdf 	nouveau fichier : res/urdf/yellow_ball.urdf

File: res/urdf/blue_bin.urdf (robot description, URDF)
Before this commit: robot blue_bin, 1 links, 0 joints
Links:
- link blue_bin: geometry collision box size=0.27 0.36 0.02; collision box size=0.27 0.36 0.02

File: res/urdf/green_bin.urdf (robot description, URDF)
Before this commit: robot green_bin, 1 links, 0 joints
Links:
- link green_bin: geometry collision box size=0.27 0.36 0.02; collision box size=0.27 0.36 0.02

File: res/urdf/green_cylinder.urdf (robot description, URDF)
Before this commit: robot orange_cup, 1 links, 0 joints
Links:
- removed link orange_cup
- added link green_cylinder, mass 0.15; collision mesh filename=package://laas_objects/res/obj/green_cyclinder.obj; visual mesh filename=package://laas_objects/res/obj/green_cyclinder.obj

File: res/urdf/table.urdf (robot description, URDF)
Before this commit: robot IKEA_table_TORSBY, 1 links, 0 joints
Links:
- link IKEA_table_TORSBY: mass 15.0 -> 60.0; geometry collision box size=0.025 0.025 0.75; collision box size=0.025 0.025 0.75
