Commit message: :ambulance: fix green cylinder

File: res/urdf/green_cylinder.urdf (robot description, URDF)
Before this commit: robot green_cylinder, 1 links, 0 joints
Links:
- link green_cylinder: geometry collision mesh filename=package://laas_objects/res/obj/green_cylinder.obj; visual mesh filename=package://laas_objects/res/obj/green_cylinder.obj
